File: ataconso/ataconso-rev-b/ataconso-rev-b.kicad_sch (KiCad schematic)
At the start: 19 parts, among them J1 Screw_Terminal_01x02, J2 Barrel_Jack_Switch, SW1 SW_SPDT, U1 NE555D, U2 NE555D

Commit message: mejorar texto
Other:
- note added: "555 derecha 1: a tierra 2: a 3 de 555 izq 3: a salida 4: a Vcc 5: a tierra por C 100n 6: a tierra por C 100n 7: a 6, a tierra por C, a Vcc por R 8: a Vcc"
- note removed: "555 derecha 1: a tierra 2: a 3 de 555 izq 3: 4: a Vcc 5: a tierra por C 100n 6: a tierra por C 100n 7: a 6, a tierra por C, a Vcc por R 8: a Vcc"
Changed lines of the file:
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@@
 		(company "piruetas SpA")
 	)
-	(text "555 derecha\n1: a tierra\n2: a 3 de 555 izq\n3:\n4: a Vcc\n5: a tierra por C 100n\n6: a tierra por C 100n\n7: a 6, a tierra por C, a Vcc por R\n8: a Vcc"
+	(text "555 derecha\n1: a tierra\n2: a 3 de 555 izq\n3: a salida\n4: a Vcc\n5: a tierra por C 100n\n6: a tierra por C 100n\n7: a 6, a tierra por C, a Vcc por R\n8: a Vcc"
 		(exclude_from_sim no)
 		(at 17.78 124.206 0)
