File: ataconso/ataconso-rev-c/ataconso-rev-c.kicad_sch (KiCad schematic)
At the start: 19 parts, among them J1 Screw_Terminal_01x02, J2 Barrel_Jack_Switch, SW1 SW_SPDT, U1 NE555D, U2 NE555D

Commit message: agregar borrador
Parts:
- removed C5: 100u, Capacitor_THT:CP_Radial_D5.0mm_P2.50mm, symbol Device:C_Polarized
- removed H1, H2: MountingHole, MountingHole:MountingHole_3.2mm_M3, symbol Mechanical:MountingHole
- removed J1: Screw_Terminal_01x02, TerminalBlock:TerminalBlock_MaiXu_MX126-5.0-02P_1x02_P5.00mm, symbol Connector:Screw_Terminal_01x02
- added C10, C3, C4, C8, C9: 100n, symbol Device:C
- added C7: 1u, symbol Device:C_Polarized
- added D1, D2: 1N5817, Diode_THT:D_DO-41_SOD81_P10.16mm_Horizontal, symbol Diode:1N5817
- added J1: Conn_02x05_Odd_Even, symbol Connector_Generic:Conn_02x05_Odd_Even
- added J2: AudioJack2_SwitchT, symbol Connector_Audio:AudioJack2_SwitchT
- added R3: 100k, symbol Device:R
- added U1: TL072, symbol Amplifier_Operational:TL072
- added U4, U5: MC78L05_SO8, Package_SO:SOIC-8_3.9x4.9mm_P1.27mm, symbol Regulator_Linear:MC78L05_SO8
- renumbered C3 to C5, C4 to C6, D1 to D3, D2 to D4, J2 to J3, R3 to R4, U1 to U2, U2 to U3
Connections:
- net GND: now also C10.1, C3.2, C4.2, C9.2, J1.3 (Pin_3), J1.4 (Pin_4), J1.5 (Pin_5), J1.6 (Pin_6), J1.7 (Pin_7), J1.8 (Pin_8), J2.1, R3.2, U1.2 (-), U1.3 (+), U4.2 (GND), U4.3 (GND), U4.6 (GND), U4.7 (GND), U5.2 (GND), U5.3 (GND), U5.6 (GND), U5.7 (GND)
- net at U3.3 (OUT): now also C7.1
- net VCC renamed +12V
- net +12V: now also C3.1, D1.1 (K), U1.8 (V+), U4.8 (IN)
- new net: C8.1, U1.6 (-), U1.7
- new net: C8.2, J2.3
- new net: C7.2, R3.1, U1.5 (+)
- new net: D1.2 (A), J1.1 (Pin_1), J1.2 (Pin_2)
- new net: D2.1 (K), J1.10 (Pin_10), J1.9 (Pin_9)
- new net +5V: C9.1, U4.1 (OUT)
- new net -12V: C4.1, D2.2 (A), U1.4 (V-), U5.8 (IN)
- new net -5V: C10.2, U5.1 (OUT)
- no-connect marks 2 -> 5
Other:
- moved on the sheet: D3, D4, J3, R4, SW1
