File: ataconso/ataconso-rev-c/ataconso-rev-c.kicad_sch (KiCad schematic)
At the start: 29 parts, among them J1 Conn_02x05_Odd_Even, J2 AudioJack2_SwitchT, J3 Barrel_Jack_Switch, SW1 SW_SPDT, U1 TL072, U2 NE555D, U3 NE555D, U4 MC78L05_SO8, U5 MC78L05_SO8

Commit message: avances en eurorack
Parts:
- removed D3: 1n4007, Diode_THT:D_DO-41_SOD81_P10.16mm_Horizontal, symbol Device:D
- removed D4: LED, LED_THT:LED_D5.0mm, symbol Device:LED
- removed J3: Barrel_Jack_Switch, Connector_BarrelJack:BarrelJack_Horizontal, symbol Connector:Barrel_Jack_Switch
- removed R4: 1k, Resistor_THT:R_Axial_DIN0207_L6.3mm_D2.5mm_P10.16mm_Horizontal, symbol Device:R
- removed SW1: SW_SPDT, parla:spdt_ssd12d00g3, symbol Switch:SW_SPDT
Connections:
- net at J1.1 (Pin_1), J1.2 (Pin_2): now also D2.1 (K); no longer D1.2 (A)
- net at J1.10 (Pin_10), J1.9 (Pin_9): now also D1.2 (A); no longer D2.1 (K)

Commit message: agregar mas avances en eurorack
Parts:
- J1: footprint (none) -> BYOM_General:IDC-Header_2x05_P2.54mm_Vertical
- J2: footprint (none) -> BYOM_General:Jack_3.5mm_QingPu_WQP-PJ398SM_Vertical
- R1, R2: footprint Resistor_THT:R_Axial_DIN0207_L6.3mm_D2.5mm_P10.16mm_Horizontal -> (none)
- U4, U5: footprint Package_SO:SOIC-8_3.9x4.9mm_P1.27mm -> (none)
Changed lines of the file:
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@@
 			)
 		)
-		(property "Footprint" ""
+		(property "Footprint" "BYOM_General:Jack_3.5mm_QingPu_WQP-PJ398SM_Vertical"
 			(at 215.9 60.96 0)
 			(hide yes)
@@
 			)
 		)
-		(property "Footprint" "Resistor_THT:R_Axial_DIN0207_L6.3mm_D2.5mm_P10.16mm_Horizontal"
+		(property "Footprint" ""
 			(at 87.122 45.72 90)
 			(hide yes)
@@
 			)
 		)
-		(property "Footprint" "Package_SO:SOIC-8_3.9x4.9mm_P1.27mm"
+		(property "Footprint" ""
 			(at 175.26 107.95 0)
 			(hide yes)
@@
 			)
 		)
-		(property "Footprint" "Resistor_THT:R_Axial_DIN0207_L6.3mm_D2.5mm_P10.16mm_Horizontal"
+		(property "Footprint" ""
 			(at 28.702 52.07 90)
 			(hide yes)
@@
 			)
 		)
-		(property "Footprint" ""
+		(property "Footprint" "BYOM_General:IDC-Header_2x05_P2.54mm_Vertical"
 			(at 120.65 135.89 0)
 			(hide yes)
@@
 			)
 		)
-		(property "Footprint" "Package_SO:SOIC-8_3.9x4.9mm_P1.27mm"
+		(property "Footprint" ""
 			(at 176.53 157.48 0)
 			(hide yes)

Commit message: borrar chip extra
Parts:
- removed C10: 100n, symbol Device:C
- removed U5: MC78L05_SO8, symbol Regulator_Linear:MC78L05_SO8

Commit message: agregar algunas huellas
Parts:
- C3, C4: footprint (none) -> Capacitor_THT:C_Disc_D3.8mm_W2.6mm_P2.50mm
Changed lines of the file:
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@@
 			)
 		)
-		(property "Footprint" ""
+		(property "Footprint" "Capacitor_THT:C_Disc_D3.8mm_W2.6mm_P2.50mm"
 			(at 77.47 128.5748 0)
 			(hide yes)
@@
 			)
 		)
-		(property "Footprint" ""
+		(property "Footprint" "Capacitor_THT:C_Disc_D3.8mm_W2.6mm_P2.50mm"
 			(at 77.47 147.0152 0)
 			(hide yes)

Commit message: actualizar potenciometros
Parts:
- RV1, RV2: footprint Potentiometer_THT:Potentiometer_Piher_PT-6-V_Vertical -> BYOM_General:POT_TH_Alps_RK09K_Single_Vertical
Changed lines of the file:
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@@
 			)
 		)
-		(property "Footprint" "Potentiometer_THT:Potentiometer_Piher_PT-6-V_Vertical"
+		(property "Footprint" "BYOM_General:POT_TH_Alps_RK09K_Single_Vertical"
 			(at 21.59 59.69 0)
 			(hide yes)
@@
 			)
 		)
-		(property "Footprint" "Potentiometer_THT:Potentiometer_Piher_PT-6-V_Vertical"
+		(property "Footprint" "BYOM_General:POT_TH_Alps_RK09K_Single_Vertical"
 			(at 88.9 27.94 0)
 			(hide yes)
