File: ataconso/ataconso-v-0-rev-c/ataconso-v-0-rev-c.kicad_pcb (KiCad board)
At the start: 2 copper layers, 20 x 100 mm, 17 parts, among them J1 Screw_Terminal_01x02, J2 Barrel_Jack_Switch, SW1 SW_SPDT, U1 NE555D, U2 NE555D

Commit message: agregar plantilla
Parts:
- removed SW1: SW_SPDT, parla:spdt_ssd12d00g3
- C5: value 100u -> 100n
- D1: value 1n4007 -> 1N5817
- D2: value LED -> 1N5817
- J1: value Screw_Terminal_01x02 -> Conn_02x05_Odd_Even; footprint TerminalBlock:TerminalBlock_MaiXu_MX126-5.0-02P_1x02_P5.00mm -> BYOM_General:IDC-Header_2x05_P2.54mm_Vertical
- J2: value Barrel_Jack_Switch -> AudioJack2_SwitchT; footprint Connector_BarrelJack:BarrelJack_Horizontal -> BYOM_General:Jack_3.5mm_QingPu_WQP-PJ398SM_Vertical
- R3: value 1k -> 100k
- RV1, RV2: footprint Potentiometer_THT:Potentiometer_Piher_PT-6-V_Vertical -> BYOM_General:POT_TH_Alps_RK09K_Single_Vertical
- U1: value NE555D -> TL072
- U2: value NE555D -> NA556; footprint Package_DIP:DIP-8_W7.62mm_Socket_LongPads -> Package_SO:SOIC-14W_7.5x9mm_P1.27mm
- moved C1 42.6 mm to (22.4, 41.9)
- moved C2 42.6 mm to (28.4, 41.9)
- moved C3 42.6 mm to (33.4, 100.9)
- moved C4 42.6 mm to (27.9, 96.9)
- moved C5 42.6 mm to (21.9, 114.9)
- moved D1 42.6 mm to (36.9, 79.0)
- moved J1 42.6 mm to (34.9, 110.9)
- moved J2 42.6 mm to (26.9, 34.9)
- moved R1 42.6 mm to (36.9, 54.9)
- moved R2 42.6 mm to (22.9, 95.9)
- moved R3 42.6 mm to (35.0, 48.9)
- moved RV1 42.6 mm to (22.9, 89.4)
- moved RV2 42.6 mm to (32.4, 89.3)
- moved U1 42.6 mm to (22.9, 55.0)
- moved U2 42.6 mm to (23.1, 70.0)
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Connections:
- C1 pad 1: Net-(U1-THRES) -> Net-(U2A-THRES)
- C2 pad 1: Net-(U1-CONT) -> Net-(U2A-CONT)
- C3 pad 1: Net-(U2-DISCH) -> +12V
- C4 pad 1: Net-(U2-CONT) -> -12V
- C5 pad 1: Net-(U2-OUT) -> Net-(U2B-DISCH)
- C5 pad 2: Net-(J1-Pin_1) -> GND
- D1 pad 1: VCC -> +12V
- D2 pad 2: VCC -> -12V
- J1 pad 1: Net-(J1-Pin_1) -> Net-(D2-K)
- J1 pad 2: GND -> Net-(D2-K)
- R1 pad 1: VCC -> +12V
- R1 pad 2: Net-(U1-DISCH) -> Net-(U2A-DISCH)
- R2 pad 2: Net-(U2-DISCH) -> Net-(U2B-DISCH)
- R3 pad 1: Net-(D2-K) -> Net-(U1B-+)
- RV1 pad 2: Net-(U1-DISCH) -> Net-(U2A-DISCH)
- RV1 pad 3: Net-(U1-THRES) -> Net-(U2A-THRES)
- RV2 pad 2: VCC -> +12V
- U1 pad 1: GND -> unconnected-(U1-Pad1)
- U1 pad 2: Net-(U1-THRES) -> GND
- U1 pad 3: Net-(U1-OUT) -> GND
- U1 pad 4: VCC -> -12V
- U1 pad 5: Net-(U1-CONT) -> Net-(U1B-+)
- U1 pad 6: Net-(U1-THRES) -> Net-(U1B--)
- U1 pad 7: Net-(U1-DISCH) -> Net-(U1B--)
- U1 pad 8: VCC -> +12V
- U2 pad 1: GND -> Net-(U2A-DISCH)
- U2 pad 2: Net-(U1-OUT) -> Net-(U2A-THRES)
- U2 pad 3: Net-(U2-OUT) -> Net-(U2A-CONT)
- U2 pad 4: VCC -> +12V
- U2 pad 5: Net-(U2-CONT) -> Net-(U2A-OUT)
- U2 pad 6: Net-(U2-DISCH) -> Net-(U2A-THRES)
- U2 pad 7: Net-(U2-DISCH) -> GND
- U2 pad 8: VCC -> Net-(U2A-OUT)
Routing:
- net VCC: track 83.8 -> 0.00 mm
- net Net-(U1-THRES): track 69.4 -> 0.00 mm
- net Net-(D1-A): track 53.5 -> 0.00 mm
- net Net-(U2-DISCH): track 49.2 -> 0.00 mm
- net Net-(U2-OUT): track 41.3 -> 0.00 mm
- net Net-(U1-DISCH): track 36.9 -> 0.00 mm
- net Net-(U2-CONT): track 22.0 -> 0.00 mm
- net Net-(U1-CONT): track 21.7 -> 0.00 mm
- net Net-(R2-Pad1): track 17.8 -> 0.00 mm
- net Net-(SW1-B): track 15.4 -> 0.00 mm
- net Net-(U1-OUT): track 14.4 -> 0.00 mm
- net Net-(D2-K): track 13.6 -> 0.00 mm
- net Net-(J1-Pin_1): track 12.2 -> 0.00 mm
- removed copper zone on B.Cu, net GND
- removed copper zone on F.Cu, net GND
