File: bloques/fuente-alimentacion/fuente-alimentacion.kicad_sch (KiCad schematic)
At the start: 7 parts, among them J2 Conn_02x05_Odd_Even, U3 L7805

Commit message: corregir bloque alimentacion, 5v ahora no es power flag
Parts:
- renumbered C10 to C4, C11 to C5, C9 to C6, J2 to J1, U3 to U1
Other:
- moved on the sheet: C6

Commit message: agregar suma-v-0-rev-a esquematico
Parts:
- renumbered C6 to C1, C4 to C2, C5 to C3, J1 to J7, U1 to U2
Changed lines of the file:
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@@
 		(in_pos_files yes)
 		(dnp no)
-		(property "Reference" "J1"
+		(property "Reference" "J7"
 			(at 40.64 60.452 0)
 			(show_name no)
@@
 			(project "suma-v-0-rev-a"
 				(path "/76d7d92c-1316-4bcb-a187-c7124ef49ded/5c6d5cb3-5959-42c3-b1d0-4c4c9800b6eb"
-					(reference "J1")
+					(reference "J7")
 					(unit 1)
 				)
@@
 		(dnp no)
 		(fields_autoplaced yes)
-		(property "Reference" "#PWR015"
+		(property "Reference" "#PWR023"
 			(at 121.92 91.44 0)
 			(hide yes)
@@
 			(project "suma-v-0-rev-a"
 				(path "/76d7d92c-1316-4bcb-a187-c7124ef49ded/5c6d5cb3-5959-42c3-b1d0-4c4c9800b6eb"
-					(reference "#PWR015")
+					(reference "#PWR023")
 					(unit 1)
 				)
@@
 		(dnp no)
 		(fields_autoplaced yes)
-		(property "Reference" "#PWR019"
+		(property "Reference" "#PWR013"
 			(at 44.45 34.29 0)
 			(hide yes)
@@
 			(project "suma-v-0-rev-a"
 				(path "/76d7d92c-1316-4bcb-a187-c7124ef49ded/5c6d5cb3-5959-42c3-b1d0-4c4c9800b6eb"
-					(reference "#PWR019")
+					(reference "#PWR013")
 					(unit 1)
 				)
@@
 		(dnp no)
 		(fields_autoplaced yes)
-		(property "Reference" "#PWR08"
+		(property "Reference" "#PWR019"
 			(at 87.63 81.28 0)
 			(hide yes)
@@
 			(project "suma-v-0-rev-a"
 				(path "/76d7d92c-1316-4bcb-a187-c7124ef49ded/5c6d5cb3-5959-42c3-b1d0-4c4c9800b6eb"
-					(reference "#PWR08")
+					(reference "#PWR019")
 					(unit 1)
 				)
@@
 		(in_pos_files yes)
 		(dnp no)
-		(property "Reference" "U1"
+		(property "Reference" "U2"
 			(at 95.25 58.42 0)
 			(show_name no)
@@
 			(project "suma-v-0-rev-a"
 				(path "/76d7d92c-1316-4bcb-a187-c7124ef49ded/5c6d5cb3-5959-42c3-b1d0-4c4c9800b6eb"
-					(reference "U1")
+					(reference "U2")
 					(unit 1)
 				)
@@
 		(dnp no)
 		(fields_autoplaced yes)
-		(property "Reference" "C5"
+		(property "Reference" "C3"
 			(at 125.73 74.9299 0)
 			(show_name no)
@@
 			(project "suma-v-0-rev-a"
 				(path "/76d7d92c-1316-4bcb-a187-c7124ef49ded/5c6d5cb3-5959-42c3-b1d0-4c4c9800b6eb"
-					(reference "C5")
+					(reference "C3")
 					(unit 1)
 				)
@@
 		(dnp no)
 		(fields_autoplaced yes)
-		(property "Reference" "#PWR017"
+		(property "Reference" "#PWR016"
 			(at 55.88 44.45 0)
 			(hide yes)
@@
 				)
 			)
+			(project "suma-v-0-rev-a"
+				(path "/76d7d92c-1316-4bcb-a187-c7124ef49ded/5c6d5cb3-5959-42c3-b1d0-4c4c9800b6eb"
+					(reference "#PWR016")
+					(unit 1)
+				)
+			)
 		)
 	)
@@
 		(dnp no)
 		(fields_autoplaced yes)
-		(property "Reference" "#PWR04"
+		(property "Reference" "#PWR017"
 			(at 60.96 81.28 0)
 			(hide yes)
@@
 			(project "suma-v-0-rev-a"
 				(path "/76d7d92c-1316-4bcb-a187-c7124ef49ded/5c6d5cb3-5959-42c3-b1d0-4c4c9800b6eb"
-					(reference "#PWR04")
+					(reference "#PWR017")
 					(unit 1)
 				)
@@
 		(dnp no)
 		(fields_autoplaced yes)
-		(property "Reference" "#PWR016"
+		(property "Reference" "#PWR015"
 			(at 55.88 34.29 0)
 			(hide yes)
@@
 			(project "suma-v-0-rev-a"
 				(path "/76d7d92c-1316-4bcb-a187-c7124ef49ded/5c6d5cb3-5959-42c3-b1d0-4c4c9800b6eb"
-					(reference "#PWR016")
+					(reference "#PWR015")
 					(unit 1)
 				)
@@
 		(dnp no)
 		(fields_autoplaced yes)
-		(property "Reference" "C6"
+		(property "Reference" "C1"
 			(at 59.055 32.1309 0)
 			(show_name no)
@@
 			(project "suma-v-0-rev-a"
 				(path "/76d7d92c-1316-4bcb-a187-c7124ef49ded/5c6d5cb3-5959-42c3-b1d0-4c4c9800b6eb"
-					(reference "C6")
+					(reference "C1")
 					(unit 1)
 				)
@@
 		(dnp no)
 		(fields_autoplaced yes)
-		(property "Reference" "#PWR01"
+		(property "Reference" "#PWR011"
 			(at 20.32 81.28 0)
 			(hide yes)
@@
 			(project "suma-v-0-rev-a"
 				(path "/76d7d92c-1316-4bcb-a187-c7124ef49ded/5c6d5cb3-5959-42c3-b1d0-4c4c9800b6eb"
-					(reference "#PWR01")
+					(reference "#PWR011")
 					(unit 1)
 				)
@@
 		(dnp no)
 		(fields_autoplaced yes)
-		(property "Reference" "#PWR014"
+		(property "Reference" "#PWR022"
 			(at 121.92 63.5 0)
 			(hide yes)
@@
 			(project "suma-v-0-rev-a"
 				(path "/76d7d92c-1316-4bcb-a187-c7124ef49ded/5c6d5cb3-5959-42c3-b1d0-4c4c9800b6eb"
-					(reference "#PWR014")
+					(reference "#PWR022")
 					(unit 1)
 				)
@@
 		(dnp no)
 		(fields_autoplaced yes)
-		(property "Reference" "#PWR07"
+		(property "Reference" "#PWR018"
 			(at 87.63 64.77 0)
 			(hide yes)
@@
 			(project "suma-v-0-rev-a"
 				(path "/76d7d92c-1316-4bcb-a187-c7124ef49ded/5c6d5cb3-5959-42c3-b1d0-4c4c9800b6eb"
-					(reference "#PWR07")
+					(reference "#PWR018")
 					(unit 1)
 				)
@@
 		(dnp no)
 		(fields_autoplaced yes)
-		(property "Reference" "#PWR020"
+		(property "Reference" "#PWR014"
 			(at 44.45 35.56 0)
 			(hide yes)
@@
 			(project "suma-v-0-rev-a"
 				(path "/76d7d92c-1316-4bcb-a187-c7124ef49ded/5c6d5cb3-5959-42c3-b1d0-4c4c9800b6eb"
-					(reference "#PWR020")
+					(reference "#PWR014")
 					(unit 1)
 				)
@@
 		(in_pos_files yes)
 		(dnp no)
-		(property "Reference" "C4"
+		(property "Reference" "C2"
 			(at 111.76 74.0409 0)
 			(show_name no)
@@
 			(project "suma-v-0-rev-a"
 				(path "/76d7d92c-1316-4bcb-a187-c7124ef49ded/5c6d5cb3-5959-42c3-b1d0-4c4c9800b6eb"
-					(reference "C4")
+					(reference "C2")
 					(unit 1)
 				)
@@
 		(dnp no)
 		(fields_autoplaced yes)
-		(property "Reference" "#PWR011"
+		(property "Reference" "#PWR021"
 			(at 107.95 91.44 0)
 			(hide yes)
@@
 			(project "suma-v-0-rev-a"
 				(path "/76d7d92c-1316-4bcb-a187-c7124ef49ded/5c6d5cb3-5959-42c3-b1d0-4c4c9800b6eb"
-					(reference "#PWR011")
+					(reference "#PWR021")
 					(unit 1)
 				)
@@
 		(dnp no)
 		(fields_autoplaced yes)
-		(property "Reference" "#PWR018"
+		(property "Reference" "#PWR012"
 			(at 22.86 43.18 0)
 			(hide yes)
@@
 			(project "suma-v-0-rev-a"
 				(path "/76d7d92c-1316-4bcb-a187-c7124ef49ded/5c6d5cb3-5959-42c3-b1d0-4c4c9800b6eb"
-					(reference "#PWR018")
+					(reference "#PWR012")
 					(unit 1)
 				)
@@
 		(dnp no)
 		(fields_autoplaced yes)
-		(property "Reference" "#PWR09"
+		(property "Reference" "#PWR020"
 			(at 95.25 91.44 0)
 			(hide yes)
@@
 			(project "suma-v-0-rev-a"
 				(path "/76d7d92c-1316-4bcb-a187-c7124ef49ded/5c6d5cb3-5959-42c3-b1d0-4c4c9800b6eb"
-					(reference "#PWR09")
-					(unit 1)
-				)
+					(reference "#PWR020")
+					(unit 1)
+				)

Commit message: agregar parla relo ataconso con bibliotecas locales
Parts:
- removed C1: 220u, Capacitor_SMD:CP_Elec_6.3x7.7, symbol Device:C_Polarized
- removed C2: 10u, Capacitor_SMD:CP_Elec_4x5.4, symbol Device:C_Polarized
- removed C3: 100n, Capacitor_SMD:C_0805_2012Metric_Pad1.18x1.45mm_HandSolder, symbol Device:C
- removed U2: L7805, Package_TO_SOT_SMD:TO-252-2, symbol Regulator_Linear:L7805
