File: plantillas/kicad/plantilla-popusintes/plantilla-popusintes.kicad_sch (KiCad schematic)
At the start: 0 parts

Commit message: agregar plantillas
Other:
- added sheet Fuente de alimentación (../../../bloques/fuente-alimentacion/fuente-alimentacion.kicad_sch)
Changed lines of the file:
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@@
   (generator_version "10.0")
   (paper "A4")
+  (sheet
+    (at 25.4 25.4)
+    (size 40.64 20.32)
+    (fields_autoplaced yes)
+    (stroke
+      (width 0.1524)
+      (type solid)
+    )
+    (fill
+      (color 0 0 0 0)
+    )
+    (property "Sheetname" "Fuente de alimentación"
+      (at 25.4 24.5219 0)
+      (effects
+        (font
+          (size 1.27 1.27)
+        )
+        (justify left bottom)
+      )
+    )
+    (property "Sheetfile" "../../../bloques/fuente-alimentacion/fuente-alimentacion.kicad_sch"
+      (at 25.4 46.0219 0)
+      (effects
+        (font
+          (size 1.27 1.27)
+        )
+        (justify left top)
+      )
+    )
+    (instances
+      (project "plantilla-popusintes"
+        (path "/76d7d92c-1316-4bcb-a187-c7124ef49ded"
+          (page "2")
+        )
+      )
+    )
+  )
   (sheet_instances
     (path "/"
-      (page "1")))
-  (embedded_fonts no))
+      (page "1")
+    )
+  )
+  (embedded_fonts no)
+)

Commit message: agregar blocks
Other:
- removed sheet Fuente de alimentación
Changed lines of the file:
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@@
   (generator_version "10.0")
   (paper "A4")
-  (sheet
-    (at 25.4 25.4)
-    (size 40.64 20.32)
-    (fields_autoplaced yes)
-    (stroke
-      (width 0.1524)
-      (type solid)
-    )
-    (fill
-      (color 0 0 0 0)
-    )
-    (property "Sheetname" "Fuente de alimentación"
-      (at 25.4 24.5219 0)
-      (effects
-        (font
-          (size 1.27 1.27)
-        )
-        (justify left bottom)
-      )
-    )
-    (property "Sheetfile" "../../../bloques/fuente-alimentacion/fuente-alimentacion.kicad_sch"
-      (at 25.4 46.0219 0)
-      (effects
-        (font
-          (size 1.27 1.27)
-        )
-        (justify left top)
-      )
-    )
-    (instances
-      (project "plantilla-popusintes"
-        (path "/76d7d92c-1316-4bcb-a187-c7124ef49ded"
-          (page "2")
-        )
-      )
-    )
-  )
   (sheet_instances
     (path "/"
