File: bibliotecas/popusintes.kicad_blocks/alimentacion-12v.kicad_block/alimentacion-12v.kicad_sch (KiCad schematic)
At the start: 3 parts, among them J1 Conn_02x05_Odd_Even

Commit message: avanzar en lcsc, huellas, stock
Other:
- title: fuente-alimentacion -> alimentacion-12v
Changed lines of the file:
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@@
 	(paper "A5")
 	(title_block
-		(title "fuente-alimentacion")
+		(title "alimentacion-12v")
 		(company "piruetas SpA")
 	)
@@
 		)
 		(instances
-			(project "fuente-alimentacion"
+			(project "alimentacion-12v"
 				(path "/18618645-9a77-4e72-b23c-6571e7d4792b"
 					(reference "J1")
@@
 		)
 		(instances
-			(project "fuente-alimentacion"
+			(project "alimentacion-12v"
 				(path "/18618645-9a77-4e72-b23c-6571e7d4792b"
 					(reference "D2")
@@
 		)
 		(instances
-			(project "fuente-alimentacion"
+			(project "alimentacion-12v"
 				(path "/18618645-9a77-4e72-b23c-6571e7d4792b"
 					(reference "#FLG01")
@@
 		)
 		(instances
-			(project "fuente-alimentacion"
+			(project "alimentacion-12v"
 				(path "/18618645-9a77-4e72-b23c-6571e7d4792b"
 					(reference "#PWR019")
@@
 		)
 		(instances
-			(project "fuente-alimentacion"
+			(project "alimentacion-12v"
 				(path "/18618645-9a77-4e72-b23c-6571e7d4792b"
 					(reference "#PWR08")
@@
 		)
 		(instances
-			(project "fuente-alimentacion"
+			(project "alimentacion-12v"
 				(path "/18618645-9a77-4e72-b23c-6571e7d4792b"
 					(reference "#FLG03")
@@
 		)
 		(instances
-			(project "fuente-alimentacion"
+			(project "alimentacion-12v"
 				(path "/18618645-9a77-4e72-b23c-6571e7d4792b"
 					(reference "D1")
@@
 		)
 		(instances
-			(project "fuente-alimentacion"
+			(project "alimentacion-12v"
 				(path "/18618645-9a77-4e72-b23c-6571e7d4792b"
 					(reference "#FLG02")
@@
 		)
 		(instances
-			(project "fuente-alimentacion"
+			(project "alimentacion-12v"
 				(path "/18618645-9a77-4e72-b23c-6571e7d4792b"
 					(reference "#PWR04")
@@
 		)
 		(instances
-			(project "fuente-alimentacion"
+			(project "alimentacion-12v"
 				(path "/18618645-9a77-4e72-b23c-6571e7d4792b"
 					(reference "#PWR01")
@@
 		)
 		(instances
-			(project "fuente-alimentacion"
+			(project "alimentacion-12v"
 				(path "/18618645-9a77-4e72-b23c-6571e7d4792b"
 					(reference "#PWR07")
@@
 		)
 		(instances
-			(project "fuente-alimentacion"
+			(project "alimentacion-12v"
 				(path "/18618645-9a77-4e72-b23c-6571e7d4792b"
 					(reference "#PWR020")
@@
 		)
 		(instances
-			(project "fuente-alimentacion"
+			(project "alimentacion-12v"
 				(path "/18618645-9a77-4e72-b23c-6571e7d4792b"
 					(reference "#PWR018")
