File: relo/relo-v-0-rev-a/relo-v-0-rev-a.kicad_sch (KiCad schematic)
At the start: 21 parts, among them J1 Conn_02x05_Odd_Even, J2 AudioJack2_SwitchT, J3 AudioJack2_SwitchT, U1 NA556, U2 TL072

Commit message: agregar parla relo ataconso con bibliotecas locales
Parts:
- J1: footprint BYOM_General:IDC-Header_2x05_P2.54mm_Vertical -> relo-v-0-rev-a:IDC-Header_2x05_P2.54mm_Vertical
- J2, J3: footprint BYOM_General:Jack_3.5mm_QingPu_WQP-PJ398SM_Vertical -> relo-v-0-rev-a:Jack_3.5mm_QingPu_WQP-PJ398SM_Vertical
- RV1, RV2: footprint BYOM_General:POT_TH_Alps_RK09K_Single_Vertical -> relo-v-0-rev-a:POT_TH_Alps_RK09K_Single_Vertical

Commit message: avanzar en lcsc, huellas, stock
Parts:
- C3, C4: footprint (none) -> Capacitor_SMD:C_0805_2012Metric_Pad1.18x1.45mm_HandSolder; LCSC (none) -> C49678
Changed lines of the file:
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@@
 			)
 		)
-		(property "Footprint" ""
+		(property "Footprint" "Capacitor_SMD:C_0805_2012Metric_Pad1.18x1.45mm_HandSolder"
 			(at 70.8152 43.18 0)
 			(hide yes)
@@
 		)
 		(property "Description" "Unpolarized capacitor"
+			(at 69.85 39.37 0)
+			(hide yes)
+			(show_name no)
+			(do_not_autoplace no)
+			(effects
+				(font
+					(size 1.27 1.27)
+				)
+			)
+		)
+		(property "LCSC" "C49678"
 			(at 69.85 39.37 0)
 			(hide yes)
@@
 			)
 		)
-		(property "Footprint" ""
+		(property "Footprint" "Capacitor_SMD:C_0805_2012Metric_Pad1.18x1.45mm_HandSolder"
 			(at 147.0152 43.18 0)
 			(hide yes)
@@
 			(at 146.05 39.37 0)
 			(hide yes)
+			(show_name no)
+			(do_not_autoplace no)
+			(effects
+				(font
+					(size 1.27 1.27)
+				)
+			)
+		)
+		(property "LCSC" "C49678"
+			(at 146.05 39.37 0)
+			(hide yes)
