File: chufe/chufe-v-0-rev-a/chufe-v-0-rev-a.kicad_pcb (KiCad board)
At the start: 0 parts

Commit message: agregar pcb-rev-a
Parts:
- added C1: 100n, Capacitor_SMD:C_0805_2012Metric, F.Cu at (59.0, 82.0)
- added C2: 100n, Capacitor_SMD:C_0805_2012Metric, F.Cu at (64.0, 82.0)
- added C3: 22u, Capacitor_SMD:CP_Elec_4x5.4, F.Cu at (81.0, 81.0)
- added D1: LED, LED_THT:LED_D3.0mm, F.Cu at (216.5, 62.5)
- added D2: LED, LED_THT:LED_D3.0mm, F.Cu at (39.0, 68.5)
- added D3: LED, LED_THT:LED_D3.0mm, F.Cu at (30.0, 68.5)
- added D4: LED, LED_THT:LED_D3.0mm, F.Cu at (34.0, 81.3)
- added J1: Conn_02x08_Odd_Even, Connector_IDC:IDC-Header_2x08_P2.54mm_Vertical, F.Cu at (60.2, 50.0)
- added J2: Conn_02x08_Odd_Even, Connector_IDC:IDC-Header_2x08_P2.54mm_Vertical, F.Cu at (92.8, 50.0)
- added J3: Conn_02x08_Odd_Even, Connector_IDC:IDC-Header_2x08_P2.54mm_Vertical, F.Cu at (125.3, 50.0)
- added J4: Conn_02x08_Odd_Even, Connector_IDC:IDC-Header_2x08_P2.54mm_Vertical, F.Cu at (157.6, 50.0)
- added J5: Conn_02x08_Odd_Even, Connector_IDC:IDC-Header_2x08_P2.54mm_Vertical, F.Cu at (190.2, 50.0)
- added J6: Barrel_Jack_Switch, Connector_BarrelJack:BarrelJack_Horizontal, F.Cu at (214.0, 51.0)
- added Q1: AO3401A, Package_TO_SOT_SMD:SOT-23, F.Cu at (203.6, 58.0)
- added R1: 2k2, Resistor_SMD:R_0805_2012Metric, F.Cu at (198.5, 63.5)
- added R2: 1k, Resistor_SMD:R_0805_2012Metric, F.Cu at (205.0, 63.5)
- added R3: 10k, Resistor_SMD:R_0805_2012Metric, F.Cu at (216.5, 68.5)
- added R4: 10k, Resistor_SMD:R_0805_2012Metric, F.Cu at (39.0, 75.0)
- added R5: 10k, Resistor_SMD:R_0805_2012Metric, F.Cu at (30.0, 75.0)
- added R6: 2k2, Resistor_SMD:R_0805_2012Metric, F.Cu at (34.0, 85.6)
- added U1: URA2412YMD-20WR3_C5369773, easyeda2kicad:PWRM-TH_YLPTEC_VRBXXXXYMD-20WR3, F.Cu at (180.0, 76.0)
- added U2: L7805, Package_TO_SOT_SMD:TO-252-2, F.Cu at (61.5, 71.9)
Routing:
- net +5V: track 0.00 -> 295.8 mm
- net +12V: track 0.00 -> 286.9 mm
- net -12V: track 0.00 -> 236.3 mm
- net /CV: track 0.00 -> 222.3 mm
- net /GATE: track 0.00 -> 185.0 mm
- net Net-(D1-A): track 0.00 -> 62.7 mm
- net Net-(Q1-D): track 0.00 -> 15.1 mm
- net Net-(Q1-G): track 0.00 -> 12.3 mm
- net Net-(D2-A): track 0.00 -> 11.3 mm
- net Net-(D3-K): track 0.00 -> 5.55 mm
- net Net-(D1-K): track 0.00 -> 5.10 mm
- net Net-(D4-K): track 0.00 -> 3.46 mm
- added copper zone on B.Cu, net GND
- added copper zone on F.Cu, net GND
Other:
- board outline added: 200 x 50 mm
- copper layers 0 -> 2
- board text added: "+12V"
- board text added: "+5V"
- board text added: "-12V"
- board text added: "chufe"
- board text added: "rev-a"
- board text added: "v0"
