File: chufebu/chufebu-v-0-rev-a/chufebu-v-0-rev-a.kicad_sch (KiCad schematic)
At the start: 10 parts, among them J1 Conn_02x08_Odd_Even, J10 Conn_01x04_Pin, J2 Conn_02x08_Odd_Even, J3 Conn_02x08_Odd_Even, J4 Conn_01x04_Pin, J5 Conn_01x04_Pin, J6 Conn_01x04_Pin, J7 Conn_02x08_Odd_Even, J8 Conn_01x04_Pin, J9 Conn_02x08_Odd_Even

Commit message: agregar borrador pcb chufe
Other:
- title: chufe-v-0 -> chufebu-v-0
- moved on the sheet: J1, J10, J2, J3, J4, J5, J6, J7, J8, J9

Commit message: agregar chufebu
Parts:
- added H1, H2: M3, MountingHole:MountingHole_3.2mm_M3, symbol Mechanical:MountingHole
- renumbered J2 to J1, J1 to J2, J5 to J4, J4 to J5, J9 to J8, J8 to J9
