File: suma/suma-v-0-rev-a/suma-v-0-rev-a.kicad_pcb (KiCad board)
At the start: 0 parts

Commit message: agregar borrador de pcb
Parts:
- added D1: D_Schottky, easyeda2kicad:SOD-123FL_L2.8-W1.8-LS3.7-R-RD, F.Cu at (46.0, 44.0)
- added D2: D_Schottky, easyeda2kicad:SOD-123FL_L2.8-W1.8-LS3.7-R-RD, F.Cu at (39.0, 44.0)
- added J1: AudioJack2_SwitchT, suma-v-0-rev-a:Jack_3.5mm_QingPu_WQP-PJ398SM_Vertical, F.Cu at (49.0, 73.5)
- added J2: AudioJack2_SwitchT, suma-v-0-rev-a:Jack_3.5mm_QingPu_WQP-PJ398SM_Vertical, F.Cu at (49.0, 89.4)
- added J3: AudioJack2_SwitchT, suma-v-0-rev-a:Jack_3.5mm_QingPu_WQP-PJ398SM_Vertical, F.Cu at (49.0, 105.4)
- added J4: AudioJack2_SwitchT, suma-v-0-rev-a:Jack_3.5mm_QingPu_WQP-PJ398SM_Vertical, F.Cu at (36.0, 121.9)
- added J5: AudioJack2_SwitchT, suma-v-0-rev-a:Jack_3.5mm_QingPu_WQP-PJ398SM_Vertical, F.Cu at (49.0, 121.9)
- added J6: Conn_02x05_Odd_Even, BYOM_General:IDC-Header_2x05_P2.54mm_Vertical, B.Cu at (37.8, 36.0)
- added R1: 100k, suma-v-0-rev-a:R0805, F.Cu at (35.0, 50.5)
- added R2: 100k, suma-v-0-rev-a:R0805, F.Cu at (35.0, 56.5)
- added R3: 100k, suma-v-0-rev-a:R0805, F.Cu at (35.0, 61.5)
- added R4: 100k, suma-v-0-rev-a:R0805, F.Cu at (51.0, 50.5)
- added R5: 100k, suma-v-0-rev-a:R0805, F.Cu at (51.0, 56.5)
- added R6: 100k, suma-v-0-rev-a:R0805, F.Cu at (51.0, 61.5)
- added R7: 1k, suma-v-0-rev-a:R0805, F.Cu at (40.0, 62.5)
- added R8: 1k, suma-v-0-rev-a:R0805, F.Cu at (45.0, 62.5)
- added RV1: 100k, suma-v-0-rev-a:POT_TH_Alps_RK09K_Single_Vertical, F.Cu at (37.5, 71.5)
- added RV2: 100k, suma-v-0-rev-a:POT_TH_Alps_RK09K_Single_Vertical, F.Cu at (37.5, 88.0)
- added RV3: 100k, suma-v-0-rev-a:POT_TH_Alps_RK09K_Single_Vertical, F.Cu at (37.5, 104.0)
- added U1: TL072, suma-v-0-rev-a:SOIC-8_L4.9-W3.9-P1.27-LS6.0-BL, F.Cu at (42.9, 54.6)
Routing:
- net Net-(J4-Pad3): track 0.00 -> 87.4 mm, vias 0 -> 2
- net Net-(J5-Pad3): track 0.00 -> 63.3 mm
- net Net-(R3-Pad1): track 0.00 -> 52.6 mm
- net Net-(R2-Pad1): track 0.00 -> 42.1 mm, vias 0 -> 2
- net Net-(U1A--): track 0.00 -> 32.9 mm
- net Net-(R1-Pad1): track 0.00 -> 29.2 mm, vias 0 -> 2
- net Net-(R6-Pad2): track 0.00 -> 20.6 mm, vias 0 -> 2
- net Net-(R4-Pad2): track 0.00 -> 20.3 mm
- net +12V: track 0.00 -> 19.9 mm
- net Net-(U1B--): track 0.00 -> 19.8 mm
- net Net-(J2-Pad3): track 0.00 -> 18.7 mm
- net Net-(J3-Pad3): track 0.00 -> 18.1 mm
- net -12V: track 0.00 -> 17.9 mm, vias 0 -> 2
- net Net-(J1-Pad3): track 0.00 -> 17.2 mm
- net Net-(D1-A): track 0.00 -> 9.49 mm
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Other:
- board outline added: 25 x 100 mm
- copper layers 0 -> 2

Commit message: agregar otra conexion faltante
Routing:
- net Net-(R4-Pad2): track 20.3 -> 31.5 mm, vias 0 -> 2
Changed lines of the file:
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@@
+	)
+	(segment
+		(start 51 49.5)
+		(end 51.5 49.5)
+		(width 0.4)
+		(layer "F.Cu")
+		(net "Net-(R4-Pad2)")
+	)
+	(segment
+		(start 48 56.5)
+		(end 49 57.5)
+		(width 0.4)
+		(layer "F.Cu")
+		(net "Net-(R4-Pad2)")
 	)
 	(segment
 		(start 49 57.5)
 		(end 51 57.5)
+		(width 0.4)
+		(layer "F.Cu")
+		(net "Net-(R4-Pad2)")
+	)
+	(segment
+		(start 51.5 49.5)
+		(end 52.5 50.5)
 		(width 0.4)
 		(layer "F.Cu")
@@
 		(net "Net-(R4-Pad2)")
 	)
+	(via
+		(at 48 56.5)
+		(size 0.6)
+		(drill 0.3)
+		(layers "F.Cu" "B.Cu")
+		(net "Net-(R4-Pad2)")
+	)
+	(via
+		(at 52.5 50.5)
+		(size 0.6)
+		(drill 0.3)
+		(layers "F.Cu" "B.Cu")
+		(net "Net-(R4-Pad2)")
+	)
+	(segment
+		(start 48 55.5)
+		(end 48 56.5)
+		(width 0.4)
+		(layer "B.Cu")
+		(net "Net-(R4-Pad2)")
+	)
+	(segment
+		(start 52.5 51)
+		(end 48 55.5)
+		(width 0.4)
+		(layer "B.Cu")
+		(net "Net-(R4-Pad2)")
+	)
+	(segment
+		(start 52.5 50.5)
+		(end 52.5 51)
+		(width 0.4)
+		(layer "B.Cu")
+		(net "Net-(R4-Pad2)")
+	)

Commit message: agregar nueva pcb
Parts:
- added C1: 100n, suma-v-0-rev-a:C0805, F.Cu at (46.6, 47.5)
- added C2: 100n, suma-v-0-rev-a:C0805, F.Cu at (33.5, 43.9)
- D1, D2: value D_Schottky -> 1N5817W; footprint easyeda2kicad:SOD-123FL_L2.8-W1.8-LS3.7-R-RD -> suma-v-0-rev-a:SOD-123FL_L2.8-W1.8-LS3.7-R-RD
- J4: value AudioJack2_SwitchT -> Conn_02x05_Odd_Even; footprint suma-v-0-rev-a:Jack_3.5mm_QingPu_WQP-PJ398SM_Vertical -> suma-v-0-rev-a:IDC-Header_2x05_P2.54mm_Vertical; moved to B.Cu
- J6: value Conn_02x05_Odd_Even -> AudioJack2_SwitchT; footprint BYOM_General:IDC-Header_2x05_P2.54mm_Vertical -> suma-v-0-rev-a:Jack_3.5mm_QingPu_WQP-PJ398SM_Vertical; moved to F.Cu
- RV1, RV2, RV3: value 100k -> A100k
- moved J4 87.6 mm to (37.6, 34.3), turned to -90 degrees
- moved J6 85.9 mm to (37.4, 121.9), turned to 0 degrees
Connections:
- J4 pad 1: GND -> Net-(D2-K)
- J4 pad 2: unconnected-(J4-Pad2) -> Net-(D2-K)
- J4 pad 3: Net-(J4-Pad3) -> GND
- J6 pad 1: Net-(D2-K) -> GND
- J6 pad 2: Net-(D2-K) -> unconnected-(J6-Pad2)
- J6 pad 3: GND -> Net-(J6-Pad3)
- R7 pad 2: Net-(J4-Pad3) -> Net-(J5-Pad3)
- R8 pad 2: Net-(J5-Pad3) -> Net-(J6-Pad3)
- RV1 pad 1: unconnected-(RV1-Pad1) -> GND
- RV1 pad 2: Net-(J1-Pad3) -> Net-(R1-Pad1)
- RV1 pad 3: Net-(R1-Pad1) -> Net-(J1-Pad3)
- RV2 pad 1: unconnected-(RV2-Pad1) -> GND
- RV2 pad 2: Net-(J2-Pad3) -> Net-(R2-Pad1)
- RV2 pad 3: Net-(R2-Pad1) -> Net-(J2-Pad3)
- RV3 pad 1: unconnected-(RV3-Pad1) -> GND
- RV3 pad 2: Net-(J3-Pad3) -> Net-(R3-Pad1)
- RV3 pad 3: Net-(R3-Pad1) -> Net-(J3-Pad3)
Routing:
- net Net-(J4-Pad3): track 87.4 -> 0.00 mm, vias 2 -> 0
- net Net-(J6-Pad3): track 0.00 -> 59.1 mm
- net GND: track 0.00 -> 15.2 mm
- net Net-(J5-Pad3): track 63.3 -> 72.7 mm, vias 0 -> 2
- net Net-(R2-Pad1): track 42.1 -> 49.3 mm, vias 2 -> 1
- net Net-(R3-Pad1): track 52.6 -> 59.1 mm
- net +12V: track 19.9 -> 23.4 mm
- net -12V: track 17.9 -> 20.8 mm
- net Net-(J3-Pad3): track 18.1 -> 20.6 mm
- net Net-(J2-Pad3): track 18.7 -> 21.2 mm
- net Net-(J1-Pad3): track 17.2 -> 19.7 mm
- net Net-(D2-K): track 9.14 -> 10.9 mm
- net Net-(D1-A): track 9.49 -> 11.1 mm
- net Net-(R1-Pad1): track 29.2 -> 28.5 mm
- added copper zone on B.Cu, net GND
- added copper zone on F.Cu, net GND

Commit message: agregar borrador suma
Parts:
- moved J5 0.71 mm to (49.5, 121.4)
- moved J6 0.58 mm to (37.7, 121.4)
- moved J1 0.50 mm to (49.5, 73.5)
- moved J2 0.50 mm to (49.5, 89.4)
- moved J3 0.50 mm to (49.5, 105.4)
- moved RV1 0.30 mm to (37.8, 71.5)
- moved RV2 0.30 mm to (37.8, 88.0)
- moved RV3 0.30 mm to (37.8, 104.0)
Routing:
- net GND: track 15.2 -> 40.7 mm, vias 0 -> 2
- net +12V: track 23.4 -> 9.57 mm
- net Net-(R4-Pad2): track 31.5 -> 41.6 mm, vias 2 -> 4
- net Net-(J6-Pad3): track 59.1 -> 68.6 mm
- net Net-(R1-Pad1): track 28.5 -> 36.0 mm, vias 2 -> 1
- net Net-(R2-Pad1): track 49.3 -> 55.6 mm, vias 1 -> 3
- net Net-(U1A--): track 32.9 -> 38.6 mm, vias 0 -> 3
- net Net-(U1B--): track 19.8 -> 24.4 mm
- net Net-(J5-Pad3): track 72.7 -> 69.4 mm, vias 2 -> 0
- net -12V: track 20.8 -> 17.6 mm, vias 2 -> 0
- net Net-(J1-Pad3): track 19.7 -> 20.8 mm
- net Net-(R6-Pad2): track 20.6 -> 19.7 mm
- net Net-(R3-Pad1): track 59.1 -> 59.5 mm, vias 0 -> 2
Other:
- board text added: "2026-10"
- board text added: "rev-a"
- board text added: "suma v0"
